File: schematic-dev/autoDistance.kicad_sch (KiCad schematic)
At the start: 6 parts, among them Q1 PN2222A, U1 HC-SR04

Commit message: StepperController Start
Parts:
- added C1: 100 uF, Capacitor_THT:CP_Radial_D8.0mm_P2.50mm, symbol Device:C
- added M1: Stepper_Motor_bipolar, symbol Motor:Stepper_Motor_bipolar
- added U2: A4988_STEPPER_MOTOR_DRIVER_CARRIER, 1-myComponents:MODULE_A4988_STEPPER_MOTOR_DRIVER_CARRIER, symbol A4988_STEPPER_MOTOR_DRIVER_CARRIER:A4988_STEPPER_MOTOR_DRIVER_CARRIER
- R1, R2, R3, R4: footprint (none) -> Resistor_THT:R_Axial_DIN0309_L9.0mm_D3.2mm_P15.24mm_Horizontal
- U1: footprint HC-SR04:XCVR_HC-SR04 -> 1-myComponents:XCVR_HC-SR04
Connections:
- net +5V: now also U2.15 (VDD)
- net ARTY: now also U2.7 (STEP), U2.8 (DIR)
- net GND: now also C1.2, U2.10 (GND), U2.16 (GND)
- new net: M1.2 (-), U2.11 (2B)
- new net: M1.1, U2.12 (2A)
- new net: M1.3, U2.13 (1A)
- new net: M1.4, U2.14 (1B)
- new net: U2.5 (~{RESET}), U2.6 (~{SLEEP})
- new net +12V: C1.1, U2.9 (VMOT)
- no-connect marks 0 -> 4
Other:
- moved on the sheet: Q1, R1, R2, R3, R4, U1
