File: schematic-files/autoDistance.kicad_sch (KiCad schematic)
At the start: 9 parts, among them M1 Stepper_Motor_bipolar, Q1 PN2222A, U1 HC-SR04, U2 A4988_STEPPER_MOTOR_DRIVER_CA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

Commit message: schematic updates
Connections:
- net +5V: now also U2.2 (MS1), U2.3 (MS2)
- removed net ARTY: Q1.1 (E), R3.2, R4.1, U2.7 (STEP), U2.8 (DIR)
- new net FPGA (Dir_Sel): U2.8 (DIR)
- new net FPGA (Recv_Pulse): R3.2, R4.1
- new net FPGA (Step_Pulse): U2.7 (STEP)
- new net FPGA (Trig_Pulse): Q1.1 (E)
- no-connect marks 4 -> 2
Other:
- moved on the sheet: C1, M1, Q1, R1, R2, R3, R4, U1, U2
